File: hardware/powerboard/powerboard.kicad_sch (KiCad schematic)
At the start: 45 parts, among them J1 BAT JST-PH 2P, J2 SERVO L, J3 SERVO R, J4 DISPLAY GC9A01, Q1 AO3401A, Q2 FS8205A, Q3 AO3401A, Q4 2N7002, Q5 AO3401A, SW1 EIN/AUS, U1 TP4054, U2 DW01A, U3 LM66100, U4 ESP32-C6-Zero

Commit message: Place the powerboard parts on a first board and render 2D and 3D views
The outline is a 45 x 30 mm placeholder until the enclosure is known, and
nothing is routed yet. The board is generated from the schematic so the
two cannot drift apart, and it shows that every part fits.

Co-Authored-By: Claude Opus 5.5 <noreply@anthropic.com>
Claude-Session: https://claude.ai/code/session_01KSMU1rRqVF3P8aDS1qPZSi
Parts:
- TP1, TP2, TP3, TP4, TP5: footprint TestPoint:TestPoint_Pad_D1.5mm -> TestPoint:TestPoint_Pad_D1.0mm
Changed lines of the file:
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@@
 			)
 		)
-		(property "Footprint" "TestPoint:TestPoint_Pad_D1.5mm"
+		(property "Footprint" "TestPoint:TestPoint_Pad_D1.0mm"
 			(at 223.52 172.72 0)
 			(effects
@@
 			)
 		)
-		(property "Footprint" "TestPoint:TestPoint_Pad_D1.5mm"
+		(property "Footprint" "TestPoint:TestPoint_Pad_D1.0mm"
 			(at 236.22 172.72 0)
 			(effects
@@
 			)
 		)
-		(property "Footprint" "TestPoint:TestPoint_Pad_D1.5mm"
+		(property "Footprint" "TestPoint:TestPoint_Pad_D1.0mm"
 			(at 248.92 172.72 0)
 			(effects
@@
 			)
 		)
-		(property "Footprint" "TestPoint:TestPoint_Pad_D1.5mm"
+		(property "Footprint" "TestPoint:TestPoint_Pad_D1.0mm"
 			(at 261.62 172.72 0)
 			(effects
@@
 			)
 		)
-		(property "Footprint" "TestPoint:TestPoint_Pad_D1.5mm"
+		(property "Footprint" "TestPoint:TestPoint_Pad_D1.0mm"
 			(at 274.32 172.72 0)
 			(effects

Commit message: Route the powerboard Rev 0.2 and add the files for a JLCPCB order
The board now has four 5 V servo ports through a TPS61023 boost, current
and voltage measurement with an INA226 on a Kelvin shunt, three analog and
two I2C ports, a THT cell connector and the outline of the shell. JLC basic
parts are used where they cost nothing in function.

The high current path (cell, reverse polarity FETs, shunt, boost, 5 V rail)
sits in one block at the front and is drawn with fixed, wide copper; the
autorouter only does signals and low current. Freerouting cannot reach pads
of parts at odd angles or next to slanted edges, so route.py rewrites the
DSN for it, tries several variants and keeps the best; maze.py closes what
is left. Labels on both sides and the KidsLab logo on the bottom.

Co-Authored-By: Claude Opus 5.5 <noreply@anthropic.com>
Claude-Session: https://claude.ai/code/session_01UqX4DjfVzW8YQJ4gc8FRQe
Parts:
- removed C8: 470u 10V, Capacitor_SMD:CP_Elec_6.3x7.7, symbol Device:C_Polarized_Small
- removed C9: 100n, Capacitor_SMD:C_0603_1608Metric, symbol Device:C_Small
- removed Q3: AO3401A, Package_TO_SOT_SMD:SOT-23, symbol Transistor_FET:AO3401A
- removed Q4: 2N7002, Package_TO_SOT_SMD:SOT-23, symbol Transistor_FET:2N7002
- removed R11, R12: 470k, Resistor_SMD:R_0603_1608Metric, symbol Device:R_Small
- removed R6: 10k, Resistor_SMD:R_0603_1608Metric, symbol Device:R_Small
- added C10, C11, C12, C13, C14: 22u, Capacitor_SMD:C_0805_2012Metric, symbol Device:C_Small
- added C15: 100n, Capacitor_SMD:C_0603_1608Metric, symbol Device:C_Small
- added J10: I2C 1, Connector_PinHeader_2.54mm:PinHeader_1x04_P2.54mm_Vertical, symbol Connector:Conn_01x04_Pin
- added J11: I2C 2, Connector_PinHeader_2.54mm:PinHeader_1x04_P2.54mm_Vertical, symbol Connector:Conn_01x04_Pin
- added J5: SERVO 3, Connector_PinHeader_2.54mm:PinHeader_1x03_P2.54mm_Vertical, symbol Connector:Conn_01x03_Pin
- added J6: SERVO 4, Connector_PinHeader_2.54mm:PinHeader_1x03_P2.54mm_Vertical, symbol Connector:Conn_01x03_Pin
- added J7: ANALOG A0, Connector_PinHeader_2.54mm:PinHeader_1x03_P2.54mm_Vertical, symbol Connector:Conn_01x03_Pin
- added J8: ANALOG A1, Connector_PinHeader_2.54mm:PinHeader_1x03_P2.54mm_Vertical, symbol Connector:Conn_01x03_Pin
- added J9: ANALOG A2, Connector_PinHeader_2.54mm:PinHeader_1x03_P2.54mm_Vertical, symbol Connector:Conn_01x03_Pin
- added L1: 1u, Inductor_SMD:L_Sunlord_MWSA0402S, symbol Device:L_Small
- added Q6: FS8205A, Package_TO_SOT_SMD:SOT-23-6, symbol powerboard:FS8205A
- added Q7: AO3401A, Package_TO_SOT_SMD:SOT-23, symbol Transistor_FET:AO3401A
- added R15: 10m, powerboard:R_1206_3216Metric_Kelvin, symbol Device:R_Shunt
- added R16, R17: 220, Resistor_SMD:R_0603_1608Metric, symbol Device:R_Small
- added R18, R19, R20: 1k, Resistor_SMD:R_0603_1608Metric, symbol Device:R_Small
- added R21, R22: 4.7k, Resistor_SMD:R_0603_1608Metric, symbol Device:R_Small
- added U5: INA226, Package_SO:TSSOP-10_3x3mm_P0.5mm, symbol Sensor_Energy:INA226
- added U6: TPS61023, Package_TO_SOT_SMD:SOT-563, symbol powerboard:TPS61023
- C7: value 47n -> 220p; LCSC (none) -> C1603
- J1: footprint Connector_JST:JST_PH_S2B-PH-SM4-TB_1x02-1MP_P2.00mm_Horizontal -> Connector_JST:JST_PH_B2B-PH-K_1x02_P2.00mm_Vertical; Kit (none) -> THT-Kit
- J2: value SERVO L -> SERVO 1
- J3: value SERVO R -> SERVO 2
- J4: footprint Connector_PinSocket_2.54mm:PinSocket_1x07_P2.54mm_Horizontal -> Connector_PinHeader_2.54mm:PinHeader_1x07_P2.54mm_Vertical; symbol Connector:Conn_01x07_Socket -> Connector:Conn_01x07_Pin
- R13, R14: LCSC (none) -> C22962
- R2: LCSC (none) -> C22775
- R4: LCSC (none) -> C23186
- R7: LCSC (none) -> C22935
- R8: value 100k -> 750k; LCSC C25803 -> C23240
- R9: value 10k -> 100k; LCSC C25804 -> C25803
- SW1: footprint Button_Switch_THT:SW_Slide_SPDT_Angled_CK_OS102011MA1Q -> powerboard:SW_Slide_SPDT_Angled_CK_OS102011MA1Q_Round
- TP4: value TP_VSERVO -> TP_V5_SERVO
- U1: value TP4054 -> TP4056; footprint Package_TO_SOT_SMD:SOT-23-5 -> Package_SO:SOIC-8-1EP_3.9x4.9mm_P1.27mm_EP2.41x3.3mm; symbol Battery_Management:LTC4054ES5-4.2 -> Battery_Management:TP4056-42-ESOP8; LCSC C668215 -> C16581
Connections:
- net Q4_D is gone; now on net GND: R9.2
- net VSERVO is gone; now on net V5_SERVO: J2.2 (Pin_2), J3.2 (Pin_2), TP4.1
- net 3V3: now also C15.1, J10.2 (Pin_2), J11.2 (Pin_2), J7.2 (Pin_2), J8.2 (Pin_2), J9.2 (Pin_2), R21.1, R22.1, U5.1 (A1), U5.2 (A0), U5.6 (VS)
- net BAT+: now also U1.5 (BAT), C10.1, L1.1, R15.4, U6.3 (VIN); no longer C7.2, Q1.2 (S), R2.1, R8.2, U1.3 (BAT)
- net BATN: now also Q6.1 (S1)
- net CHRG_N: now also U1.7 (~{CHRG}); no longer U1.1 (~{CHRG})
- net DW_OC: now also Q6.4 (G2)
- net DW_OD: now also Q6.6 (G1)
- net FET_D: now also Q6.2 (D), Q6.5 (D)
- net GND: now also U1.1 (TEMP), U1.3 (GND), U1.9 (EPAD), C10.2, C11.2, C12.2, C13.2, C14.2, C15.2, J10.1 (Pin_1), J11.1 (Pin_1), J5.3 (Pin_3), J6.3 (Pin_3), J7.1 (Pin_1), J8.1 (Pin_1), J9.1 (Pin_1), Q6.3 (S2), U5.7 (GND), U6.4 (GND); no longer U1.2 (GND)
- net J_BATP: now also Q7.3 (D)
- net PROG: now also U1.2 (PROG); no longer U1.5 (PROG)
- net Q1_G: now also Q7.1 (G)
- net SERVO_EN: now also U4.13 (GPIO15), U6.2 (EN); no longer U4.6 (GPIO2)
- net VSYS: now also U1.8 (CE)
- net SERVO3: now reaches U4.10 (TX/GPIO16)
- net SERVO3: now also R16.1
- net SERVO4: now reaches U4.11 (RX/GPIO17)
- net SERVO4: now also R17.1
- net I2C_SDA: now reaches U4.12 (GPIO14)
- net I2C_SDA: now also J10.3 (Pin_3), J11.3 (Pin_3), R21.2, U5.4 (SDA)
- net I2C_SCL: now reaches U4.18 (GPIO22)
- net I2C_SCL: now also J10.4 (Pin_4), J11.4 (Pin_4), R22.2, U5.5 (SCL)
- net CHRG_IO renamed A1_IO
- net A1_IO: now also R19.2
- net SERVO_G renamed V5_SERVO
- net V5_SERVO: now also C11.1, C12.1, C13.1, C14.1, J5.2 (Pin_2), J6.2 (Pin_2), U6.6 (VOUT); no longer R9.1
- net SERVO_L renamed SERVO1
- net SERVO_L_S renamed SERVO1_S
- net SERVO_R renamed SERVO2
- net SERVO_R_S renamed SERVO2_S
- net VBAT_SENSE renamed A0_IO
- net A0_IO: now also R18.2
- new net A0: J7.3 (Pin_3), R18.1
- new net A1: J8.3 (Pin_3), R19.1
- new net A2: J9.3 (Pin_3), R20.1
- new net A2_IO: R20.2, U4.6 (GPIO2)
- new net BAT_CELL: Q1.2 (S), Q7.2 (S), R15.1, R2.1
- new net BOOST_FB: C7.2, R8.2, R9.1, U6.1 (FB)
- new net BOOST_SW: L1.2, U6.5 (SW)
- new net SENSE_N: R15.3, U5.8 (Vbus), U5.9 (Vin-)
- new net SENSE_P: R15.2, U5.10 (Vin+)
- new net SERVO3_S: J5.1 (Pin_1), R16.2
- new net SERVO4_S: J6.1 (Pin_1), R17.2
- no-connect marks 9 -> 6
Other:
- note added: "Analog 3V3"
- note added: "Display, per Kabel"
- note added: "Ein/Aus (Q5) + Power Path (LM66100)"
- note added: "I2C 3V3"
- note added: "Lader TP4056, 235 mA"
- note added: "Schutz: DW01A + 2x FS8205A"
- note added: "Servo-Ports"
- note added: "Servo-Schiene 5 V (TPS61023, GPIO15 schaltet)"
- note added: "Strom + Spannung: INA226"
- note removed: "Akkumessung GPIO0"
- note removed: "Display, direkt gesteckt"
- note removed: "Ein/Aus (Q5) + Power Path (LM66100, CE fest auf GND)"
- note removed: "Lader TP4054, 200 mA"
- note removed: "Schutz: DW01A + FS8205A (BATN nur hier und an J1)"
- note removed: "Servo-Schiene (GPIO2 schaltet, nur aus dem Akku)"
- moved on the sheet: C1, C2, C3, C4, C5, C6, C7, D1, H1, H2, J1, J2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
